File: PCB/Ibanez_FL-9.kicad_sch (KiCad schematic)
At the start: 155 parts, among them J1 INPUT, J2 OUTPUT, J3 EXT_DC, Q101 2SC2458GR, Q102 2SC2458GR, Q103 2SK44SPC, Q104 2SC2458GR, Q105 2SC2458GR, Q106 2SC2458GR, Q107 2SA1048Y/GR, Q108A1001 2SC1583F, Q108B1001 2SC1583F, Q109 2SC2458GR, SW1 NORMAL/EFFECT, U101 TL022, U102 TL022, U103 TL022, U104 MN3207, U105 MN3102, U106 LM78L05_TO92

Commit message: update pcb layout
Parts:
- C103, C105: footprint Capacitor_THT:C_Rect_L7.0mm_W2.5mm_P5.00mm -> Capacitor_THT:C_Rect_L7.0mm_W2.0mm_P5.00mm
- D103, D104, D107: footprint Diode_THT:D_DO-35_SOD27_P7.62mm_Horizontal -> Diode_THT:D_T-1_P2.54mm_Vertical_KathodeUp
Connections:
- net +5V: now also R114.1, R147.1; no longer R114.2, R147.2
- net 4.5v: now also R102.2, R130.2; no longer R102.1, R130.1
- net CP4: now also R103.2, R105.1; no longer R103.1, R105.2
- net CP5: now also R110.1; no longer R110.2
- net CP9: now also R145.1; no longer R145.2
- net GND: now also R115.2; no longer R115.1
- net at C105.2: now also R104.1; no longer R104.2
- net at C106.1, R111.2: now also R110.2; no longer R110.1
- net at C102.1, U101.6 (-): now also R103.1, R104.2; no longer R103.2, R104.1
- net at R101.2: now also R102.1, U101.5 (+); no longer C101.2
- net at RV102.3: now also R115.1; no longer R115.2
- net at C104.1: now also R105.2; no longer R105.1
- net at C120.2: now also R131.1; no longer R131.2
- net at JP3.1 (A), R132.2: now also R131.2; no longer R131.1
- net at D101.2 (A), D102.1 (K): now also R108.2; no longer R108.1
- net at C104.2, R107.2, U102.6 (-): now also R108.1, R109.1; no longer R108.2, R109.2
- net at RV103.1: now also R109.2; no longer R109.1
- net at C127.2, Q107.3 (B), R146.2: now also R147.2; no longer R147.1
- net at RV102.1: now also R114.2; no longer R114.1
- net at Q107.2 (C), R148.1: now also R145.2; no longer R145.1
- net at U101.3 (+): now also R130.1; no longer R130.2
- new net: C101.2, R101.1
Other:
- note added: "BATTERY CHECKER"
- note added: "CLOCK VCO AND DRIVER"
- note added: "LOW FREQUENCY OSCILLATOR"
- note added: "LOW-PASS -12dB/OCT"
- note added: "LOW-PASS -24dB/OCT"
- note added: "MIXER AND CLAMPER"
- note added: "MIXER AND DE-EMPHASIS"
- note added: "POWER: VOLTAGE REGULATION"
- note added: "PRE-EMPHASIS"
- note added: "SWITCHING DRIVER"
- note removed: "DELAY OUTPUT FILTER"
- note removed: "INPUT BUFFER AMP"
- note removed: "LED DRIVER"
- note removed: "LEVEL CONVERTER"
- note removed: "NORMAL/EFFECT TOGGLE FLIP-FLOP"
- note removed: "OUTPUT SUMMING AMP"
- note removed: "POWER"
- note removed: "REGENERATIVE SUM AMP"
- note removed: "SWEEP OSCILLATOR"
- moved on the sheet: R101, R102, R103, R104, R105, R108, R109, R110, R114, R115, R130, R131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

Commit message: update pcb layout
Parts:
- added R143: 1M, Resistor_THT:R_Axial_DIN0204_L3.6mm_D1.6mm_P2.54mm_Vertical, symbol Device:R_Small
- C113, C119: footprint Capacitor_THT:C_Rect_L7.0mm_W2.5mm_P5.00mm -> Capacitor_THT:C_Rect_L7.0mm_W2.0mm_P5.00mm
- Q101, Q102, Q103, Q104, Q105, Q106, Q107, Q108A1001, Q108B1001, Q109: footprint Package_TO_SOT_THT:TO-92_Inline -> Package_TO_SOT_THT:TO-92Flat
Connections:
- net 4.5v: now also R106.2, R120.2; no longer R106.1, R120.1
- net CP12: now also R123.1; no longer R123.2
- net CP15: now also R129.2; no longer R129.1
- net CP4: now also R127.1; no longer R127.2
- net GND: now also R123.2; no longer R123.1
- net at C202.1, Q105.2 (C), R133.2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: now also R143.2; no longer Q106.3 (B)
- net at C118.1, R126.1, R128.2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: now also R127.2, R129.1; no longer R127.1, R129.2
- net at U102.3 (+): now also R120.1; no longer R120.2
- net at U102.5 (+): now also R106.1; no longer R106.2
- new net: Q106.3 (B), R143.1
Other:
- moved on the sheet: D103, R106, R120, R123, R127, R129, R133

Commit message: pcb layout v1.0
Parts:
- BT1: footprint Battery:BatteryHolder_MPD_BA9VPC_1xPP3 -> (none)
- C111: footprint Capacitor_THT:C_Rect_L7.0mm_W2.5mm_P5.00mm -> Capacitor_THT:C_Rect_L7.0mm_W2.0mm_P5.00mm
- C112: value 0.001uf CER -> 0.001uf FILM; footprint Capacitor_THT:C_Disc_D3.0mm_W2.0mm_P2.50mm -> Capacitor_THT:C_Rect_L7.0mm_W2.0mm_P5.00mm
- C129: value 0.01uf -> 0.01uf FILM; footprint Capacitor_THT:C_Disc_D3.0mm_W2.0mm_P2.50mm -> Capacitor_THT:C_Rect_L7.0mm_W2.0mm_P5.00mm
- D1: footprint LED_THT:LED_D3.0mm_Clear -> (none)
- D105: footprint Diode_THT:D_DO-15_P2.54mm_Vertical_KathodeUp -> Diode_THT:D_T-1_P2.54mm_Vertical_KathodeUp
- RV1, RV2, RV3, RV4: footprint Potentiometer_THT:Potentiometer_ACP_CA6-H2,5_Horizontal -> (none)
- SW1: footprint Button_Switch_THT:SW_PUSH-12mm -> (none)
Connections:
- net +9V: now also R134.1, R135.1; no longer R134.2, R135.2
- net GND: now also R140.2; no longer R140.1
- net at C129.2, JP13.2 (B), U103.1: now also R155.2; no longer R155.1
- net at C202.1, Q105.2 (C), R133.2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: now also R134.2; no longer R134.1
- net at C110.2: now also R117.1; no longer R117.2
- net at C201.2, Q104.2 (C), R201.1: now also R135.2; no longer R135.1
- net at C122.1, C123.1, C124.2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: now also R141.1; no longer R141.2
- net at C112.1, U102.2 (-): now also R118.2; no longer R118.1
- net at C128.1, Q108B1001.3 (B), R151.2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: now also R149.2; no longer R149.1
- net at C111.2, R119.2: now also R117.2, R118.1; no longer R117.1, R118.2
- net at JP11.1 (A): now also R141.2; no longer R141.1
- net at Q108A1001.2 (C), Q108A1001.3 (B), R150.1: now also R149.1; no longer R149.2
- net at C131.2, JP6.2 (B), U103.7: now also R156.1; no longer R156.2
- net at R138.1, R139.1: now also R140.1; no longer R140.2
- new net: R155.1, R156.2, U103.3 (+)
Other:
- moved on the sheet: R117, R118, R134, R135, R140, R141, R149, R155, R156
