File: PCB/Ibanez_FL-9.kicad_sch (KiCad schematic)
At the start: 156 parts, among them IC101 TL022, IC102 TL022, IC103 TL022, IC104 MN3207, IC105 MN3102, IC106 LM78L05_TO92, J1 INPUT, J2 OUTPUT, J3 EXT_DC, Q101 2SC2458GR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

Commit message: update testpoints on bot silk; fix spelling
Parts:
- renumbered U101 to IC101, U102 to IC102, U103 to IC103
Changed lines of the file:
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@@
   (title_block
     (title "Ibanez_FL-9_Flanger_Pedal MP-FL0601")
-    (date "2022-11-29")
+    (date "2022-12-04")
     (rev "1.0.0")
     (company "Cedar Grove Studios")
@@
     (effects (font (size 1.524 1.524) (thickness 0.254) bold italic) (justify left bottom))
   )
-  (label "CP15" (at 330.835 43.815 0)
+  (label "CP15" (at 330.835 42.545 0)
     (effects (font (size 1.524 1.524) (thickness 0.254) bold italic) (justify left bottom))
   )
@@
   (symbol (lib_id "Amplifier_Operational:TL072") (at 196.215 171.45 0) (unit 3)
     (in_bom yes) (on_board yes)
-    (property "Reference" "U102" (id 0) (at 194.31 170.5415 0)
+    (property "Reference" "IC102" (id 0) (at 194.31 170.5415 0)
       (effects (font (size 1.27 1.27)) (justify left))
     )
@@
   (symbol (lib_id "Amplifier_Operational:TL072") (at 208.915 170.815 0) (unit 3)
     (in_bom yes) (on_board yes)
-    (property "Reference" "U103" (id 0) (at 207.01 169.9065 0)
+    (property "Reference" "IC103" (id 0) (at 207.01 169.9065 0)
       (effects (font (size 1.27 1.27)) (justify left))
     )
@@
   (symbol (lib_id "Amplifier_Operational:TL072") (at 183.515 172.085 0) (unit 3)
     (in_bom yes) (on_board yes)
-    (property "Reference" "U101" (id 0) (at 181.61 171.1765 0)
+    (property "Reference" "IC101" (id 0) (at 181.61 171.1765 0)
       (effects (font (size 1.27 1.27)) (justify left))
     )
@@
       (reference "IC101") (unit 2) (value "TL022") (footprint "Package_DIP:DIP-8_W7.62mm")
     )
+    (path "/c0238134-b46d-42a1-9fdb-86790b8a110e"
+      (reference "IC101") (unit 3) (value "TL022") (footprint "Package_DIP:DIP-8_W7.62mm")
+    )
     (path "/fc8ffd4f-592d-4600-af07-01b564606849"
       (reference "IC102") (unit 1) (value "TL022") (footprint "Package_DIP:DIP-8_W7.62mm")
@@
       (reference "IC102") (unit 2) (value "TL022") (footprint "Package_DIP:DIP-8_W7.62mm")
     )
+    (path "/37322642-a9e8-4b7a-994e-382297571ca4"
+      (reference "IC102") (unit 3) (value "TL022") (footprint "Package_DIP:DIP-8_W7.62mm")
+    )
     (path "/156cc437-73f9-4b3d-899d-c1d51a8c376d"
       (reference "IC103") (unit 1) (value "TL022") (footprint "Package_DIP:DIP-8_W7.62mm")
@@
       (reference "IC103") (unit 2) (value "TL022") (footprint "Package_DIP:DIP-8_W7.62mm")
     )
+    (path "/80bbc5b6-fa99-4be6-8706-175bfe844748"
+      (reference "IC103") (unit 3) (value "TL022") (footprint "Package_DIP:DIP-8_W7.62mm")
+    )
     (path "/ed34a539-454e-41b2-957f-a6259baf48fe"
       (reference "IC104") (unit 1) (value "MN3207") (footprint "Package_DIP:DIP-8_W7.62mm")
@@
       (reference "SW1") (unit 1) (value "NORMAL/EFFECT") (footprint "")
     )
-    (path "/c0238134-b46d-42a1-9fdb-86790b8a110e"
-      (reference "U101") (unit 3) (value "TL022") (footprint "Package_DIP:DIP-8_W7.62mm")
-    )
-    (path "/37322642-a9e8-4b7a-994e-382297571ca4"
-      (reference "U102") (unit 3) (value "TL022") (footprint "Package_DIP:DIP-8_W7.62mm")
-    )
-    (path "/80bbc5b6-fa99-4be6-8706-175bfe844748"
-      (reference "U103") (unit 3) (value "TL022") (footprint "Package_DIP:DIP-8_W7.62mm")
-    )
   )
