File: PCB/Ibanez_FL-9.kicad_pcb (KiCad board)
At the start: 2 copper layers, 60 x 77 mm, 147 parts, among them J3 EXT_DC, Q101 2SC2458GR, Q102 2SC2458GR, Q103 2SK44SPC, Q104 2SC2458GR, Q105 2SC2458GR, Q106 2SC2458GR, Q107 2SA1048Y/GR, Q108 2SC1583F, Q109 2SC2458GR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

Commit message: update schematic, guide, and docs
Parts:
- renumbered U101 to IC101, U102 to IC102, U103 to IC103, U104 to IC104, U105 to IC105, U106 to IC106
Connections:
- IC101 pad 4: GND -> (no net)
- IC101 pad 8: +9V -> (no net)
- IC102 pad 4: GND -> (no net)
- IC102 pad 8: +9V -> (no net)
- IC103 pad 4: GND -> (no net)
- IC103 pad 8: +5V -> (no net)
Changed lines of the file:
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@@
   (title_block
     (title "Ibanez_FL-9_Flanger_Pedal MP-FL0601")
-    (date "2022-11-24")
+    (date "2022-11-26")
     (rev "v02")
     (company "Cedar Grove Studios")
@@
   (net 80 "Net-(JP7-Pad2)")
   (net 81 "Net-(JP16-Pad2)")
-  (net 82 "Net-(U104-Pad2)")
+  (net 82 "Net-(IC104-Pad2)")
   (net 83 "/CP1")
-  (net 84 "unconnected-(U105-Pad6)")
+  (net 84 "unconnected-(IC105-Pad6)")
   (net 85 "Net-(BT1-Pad1)")
   (net 86 "Net-(J1-PadT)")
@@
     (property "Sheetname" "")
     (attr through_hole)
-    (fp_text reference "U101" (at 2.1 -1.9) (layer "F.SilkS")
+    (fp_text reference "IC101" (at 2.1 -1.9) (layer "F.SilkS")
       (effects (font (size 0.5 0.5) (thickness 0.1)))
     )
@@
     (pad "3" thru_hole oval locked (at 0 5.08) (size 1.6 1.6) (drill 0.8) (layers *.Cu *.Mask)
       (net 90 "Net-(R130-Pad1)") (pinfunction "+") (pintype "input"))
-    (pad "4" thru_hole oval locked (at 0 7.62) (size 1.6 1.6) (drill 0.8) (layers *.Cu *.Mask)
-      (net 13 "GND") (pinfunction "V-") (pintype "power_in"))
+    (pad "4" thru_hole oval locked (at 0 7.62) (size 1.6 1.6) (drill 0.8) (layers *.Cu *.Mask))
     (pad "5" thru_hole oval locked (at 7.62 7.62) (size 1.6 1.6) (drill 0.8) (layers *.Cu *.Mask)
       (net 89 "Net-(R101-Pad2)") (pinfunction "+") (pintype "input"))
@@
     (pad "7" thru_hole oval locked (at 7.62 2.54) (size 1.6 1.6) (drill 0.8) (layers *.Cu *.Mask)
       (net 4 "/CP4") (pintype "output"))
-    (pad "8" thru_hole oval locked (at 7.62 0) (size 1.6 1.6) (drill 0.8) (layers *.Cu *.Mask)
-      (net 43 "+9V") (pinfunction "V+") (pintype "power_in"))
+    (pad "8" thru_hole oval locked (at 7.62 0) (size 1.6 1.6) (drill 0.8) (layers *.Cu *.Mask))
     (model "${KICAD6_3DMODEL_DIR}/Package_DIP.3dshapes/DIP-8_W7.62mm.wrl"
       (offset (xyz 0 0 0))
@@
     (property "Sheetname" "")
     (attr through_hole)
-    (fp_text reference "U103" (at -0.3 -2.1) (layer "F.SilkS")
+    (fp_text reference "IC103" (at -0.3 -2.1) (layer "F.SilkS")
       (effects (font (size 0.5 0.5) (thickness 0.1)))
     )
@@
     (pad "3" thru_hole oval locked (at 0 5.08) (size 1.6 1.6) (drill 0.8) (layers *.Cu *.Mask)
       (net 92 "Net-(R155-Pad1)") (pinfunction "+") (pintype "input"))
-    (pad "4" thru_hole oval locked (at 0 7.62) (size 1.6 1.6) (drill 0.8) (layers *.Cu *.Mask)
-      (net 13 "GND") (pinfunction "V-") (pintype "power_in"))
+    (pad "4" thru_hole oval locked (at 0 7.62) (size 1.6 1.6) (drill 0.8) (layers *.Cu *.Mask))
     (pad "5" thru_hole oval locked (at 7.62 7.62) (size 1.6 1.6) (drill 0.8) (layers *.Cu *.Mask)
       (net 42 "Net-(C132-Pad1)") (pinfunction "+") (pintype "input"))
@@
     (pad "7" thru_hole oval locked (at 7.62 2.54) (size 1.6 1.6) (drill 0.8) (layers *.Cu *.Mask)
       (net 40 "Net-(C130-Pad1)") (pintype "output"))
-    (pad "8" thru_hole oval locked (at 7.62 0) (size 1.6 1.6) (drill 0.8) (layers *.Cu *.Mask)
-      (net 44 "+5V") (pinfunction "V+") (pintype "power_in"))
+    (pad "8" thru_hole oval locked (at 7.62 0) (size 1.6 1.6) (drill 0.8) (layers *.Cu *.Mask))
     (model "${KICAD6_3DMODEL_DIR}/Package_DIP.3dshapes/DIP-8_W7.62mm.wrl"
       (offset (xyz 0 0 0))
@@
     (property "Sheetname" "")
     (attr through_hole)
-    (fp_text reference "U105" (at 7.1 -2.4 180) (layer "F.SilkS")
+    (fp_text reference "IC105" (at 7.1 -2.4 180) (layer "F.SilkS")
       (effects (font (size 0.5 0.5) (thickness 0.1)))
     )
@@
       (net 44 "+5V") (pinfunction "VDD") (pintype "power_in"))
     (pad "2" thru_hole oval locked (at 0 2.54 90) (size 1.6 1.6) (drill 0.8) (layers *.Cu *.Mask)
-      (net 82 "Net-(U104-Pad2)") (pinfunction "CP1") (pintype "output"))
+      (net 82 "Net-(IC104-Pad2)") (pinfunction "CP1") (pintype "output"))
     (pad "3" thru_hole oval locked (at 0 5.08 90) (size 1.6 1.6) (drill 0.8) (layers *.Cu *.Mask)
       (net 13 "GND") (pinfunction "GND") (pintype "power_in"))
@@
       (net 35 "Net-(C126-Pad1)") (pinfunction "OX3") (pintype "input"))
     (pad "6" thru_hole oval locked (at 7.62 5.08 90) (size 1.6 1.6) (drill 0.8) (layers *.Cu *.Mask)
-      (net 84 "unconnected-(U105-Pad6)") (pinfunction "OX2") (pintype "input+no_connect"))
+      (net 84 "unconnected-(IC105-Pad6)") (pinfunction "OX2") (pintype "input+no_connect"))
     (pad "7" thru_hole oval locked (at 7.62 2.54 90) (size 1.6 1.6) (drill 0.8) (layers *.Cu *.Mask)
       (net 36 "/CP9") (pinfunction "OX1") (pintype "input"))
@@
     (property "Sheetname" "")
     (attr through_hole)
-    (fp_text reference "U104" (at 5.1 -2.4 180) (layer "F.SilkS")
+    (fp_text reference "IC104" (at 5.1 -2.4 180) (layer "F.SilkS")
       (effects (font (size 0.5 0.5) (thickness 0.1)))
     )
@@
       (net 13 "GND") (pinfunction "GND") (pintype "power_in"))
     (pad "2" thru_hole oval locked (at 0 2.54 270) (size 1.6 1.6) (drill 0.8) (layers *.Cu *.Mask)
-      (net 82 "Net-(U104-Pad2)") (pinfunction "CP1") (pintype "input"))
+      (net 82 "Net-(IC104-Pad2)") (pinfunction "CP1") (pintype "input"))
     (pad "3" thru_hole oval locked (at 0 5.08 270) (size 1.6 1.6) (drill 0.8) (layers *.Cu *.Mask)
       (net 15 "Net-(C108-Pad2)") (pinfunction "IN") (pintype "input"))
@@
     (property "Sheetname" "")
     (attr through_hole)
-    (fp_text reference "U102" (at 8.2 -2.2) (layer "F.SilkS")
+    (fp_text reference "IC102" (at 8.2 -2.2) (layer "F.SilkS")
       (effects (font (size 0.5 0.5) (thickness 0.1)))
     )
@@
     (pad "3" thru_hole oval locked (at 0 5.08) (size 1.6 1.6) (drill 0.8) (layers *.Cu *.Mask)
       (net 88 "Net-(R120-Pad1)") (pinfunction "+") (pintype "input"))
-    (pad "4" thru_hole oval locked (at 0 7.62) (size 1.6 1.6) (drill 0.8) (layers *.Cu *.Mask)
-      (net 13 "GND") (pinfunction "V-") (pintype "power_in"))
+    (pad "4" thru_hole oval locked (at 0 7.62) (size 1.6 1.6) (drill 0.8) (layers *.Cu *.Mask))
     (pad "5" thru_hole oval locked (at 7.62 7.62) (size 1.6 1.6) (drill 0.8) (layers *.Cu *.Mask)
       (net 73 "Net-(R106-Pad1)") (pinfunction "+") (pintype "input"))
@@
     (pad "7" thru_hole oval locked (at 7.62 2.54) (size 1.6 1.6) (drill 0.8) (layers *.Cu *.Mask)
       (net 49 "/CP5") (pintype "output"))
-    (pad "8" thru_hole oval locked (at 7.62 0) (size 1.6 1.6) (drill 0.8) (layers *.Cu *.Mask)
-      (net 43 "+9V") (pinfunction "V+") (pintype "power_in"))
+    (pad "8" thru_hole oval locked (at 7.62 0) (size 1.6 1.6) (drill 0.8) (layers *.Cu *.Mask))
     (model "${KICAD6_3DMODEL_DIR}/Package_DIP.3dshapes/DIP-8_W7.62mm.wrl"
       (offset (xyz 0 0 0))
@@
     (property "Sheetname" "")
     (attr through_hole)
-    (fp_text reference "U106" (at -1.53 1.74) (layer "F.SilkS")
+    (fp_text reference "IC106" (at -1.53 1.74) (layer "F.SilkS")
       (effects (font (size 0.5 0.5) (thickness 0.1)))
     )
